File: hardware/KiCad/FC_v1.0/FC-power-section.kicad_sch (KiCad schematic)
At the start: 33 parts, among them J1 SM06B-GHS-TB, U2 TPS2113ADRBR, U3 TPS62130ARGTR, U4 TPS7A2133PQWDRBRQ1

Commit message: board_testing_docs
Parts:
- U2: footprint FC-FootprintLib:TPS2113A -> FC-FootprintLib:TPS2113ADRBR; Supplier Link 2 https://jlcpcb.com/parts/componentSearch?searchTxt=TPS2113A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 -> https://jlcpcb.com/partdetail/TexasInstruments-TPS2113ADRBR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
Changed lines of the file:
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@@
 			)
 		)
-		(property "Footprint" "FC-FootprintLib:TPS2113A"
+		(property "Footprint" "FC-FootprintLib:TPS2113ADRBR"
 			(at 166.37 92.71 0)
 			(effects
@@
 			)
 		)
-		(property "Supplier Link 2" "https://jlcpcb.com/parts/componentSearch?searchTxt=TPS2113ADRBR"
+		(property "Supplier Link 2" "https://jlcpcb.com/partdetail/TexasInstruments-TPS2113ADRBR/C354512"
 			(at 232.156 106.68 0)
 			(effects
