File: hardware/KiCad/FC_v1.0/FC-proto.kicad_pcb (KiCad board)
At the start: 4 copper layers, 56 x 46 mm, 135 parts, among them J1 SM06B-GHS-TB, J10 PAD_OUT, J11 PAD_OUT, J12 Conn_01x05, J13 Conn_01x05, J2 MEM2061-01-188-00-A, J3 USB4105-GF-A, J4 Conn_ARM_SWD_TagConnect_TC203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, J5 SM06B-GHS-TB, J6 SM04B-GHS-TB, J7 SM06B-GHS-TB, J8 SM06B-GHS-TB, J9 SM04B-GHS-TB, Q1 AO3400A, SW1 PCM12SMTRFC, U1 STM32H743ZIT6, U2 TPS2113ADRBR, U3 TPS62130ARGTR, U4 TPS7A2133PQWDRBRQ1, U5 ICM-40609-D, U6 MMC5983MA, U7 BMP390, U8 TPD2EUSB30A, Y2 16MHz

Commit message: board_testing_docs
Parts:
- U2: footprint FC-FootprintLib:TPS2113A -> FC-FootprintLib:TPS2113ADRBR
